File: alarm_panel_breakout/12v_Buffered_Input.kicad_sch (KiCad schematic)
At the start: 5 parts

Commit message: alarm panel initial layout
Parts:
- C17: renamed from C?; footprint (none) -> Capacitor_SMD:C_0603_1608Metric
- gave numbers to parts that had none: 4
Connections:
- net Output: now also C17.1
Other:
- moved on the sheet: C17
Changed lines of the file:
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@@
   (junction (at 123.19 77.47) (diameter 0) (color 0 0 0 0)
+  )
+  (junction (at 143.51 72.39) (diameter 0) (color 0 0 0 0)
+  )
+  (wire (pts (xy 143.51 72.39) (xy 132.08 72.39))
+    (stroke (width 0) (type default) (color 0 0 0 0))
   )
   (wire (pts (xy 121.92 77.47) (xy 123.19 77.47))
@@
     (stroke (width 0) (type default) (color 0 0 0 0))
   )
-  (wire (pts (xy 146.05 72.39) (xy 132.08 72.39))
+  (wire (pts (xy 146.05 72.39) (xy 143.51 72.39))
     (stroke (width 0) (type default) (color 0 0 0 0))
   )
@@
   (symbol (lib_id "power:GND") (at 123.19 85.09 0)
     (in_bom yes) (on_board yes) (fields_autoplaced)
-    (property "Reference" "#PWR?" (id 0) (at 123.19 91.44 0)
+    (property "Reference" "#PWR0201" (id 0) (at 123.19 91.44 0)
       (effects (font (size 1.27 1.27)) hide)
     )
@@
   (symbol (lib_id "Device:R") (at 118.11 77.47 90)
     (in_bom yes) (on_board yes) (fields_autoplaced)
-    (property "Reference" "R?" (id 0) (at 118.11 72.4875 90))
+    (property "Reference" "R44" (id 0) (at 118.11 72.4875 90))
     (property "Value" "1K" (id 1) (at 118.11 75.2626 90))
     (property "Footprint" "Resistor_SMD:R_0603_1608Metric" (id 2) (at 118.11 79.248 90)
@@
     (pin "2")
   )
-  (symbol (lib_id "Device:C") (at 144.78 76.2 0)
+  (symbol (lib_id "Device:C") (at 143.51 76.2 0)
     (in_bom yes) (on_board yes) (fields_autoplaced)
-    (property "Reference" "C?" (id 0) (at 147.701 75.2915 0)
+    (property "Reference" "C17" (id 0) (at 146.431 75.2915 0)
       (effects (font (size 1.27 1.27)) (justify left))
     )
-    (property "Value" "C" (id 1) (at 147.701 78.0666 0)
+    (property "Value" "C" (id 1) (at 146.431 78.0666 0)
       (effects (font (size 1.27 1.27)) (justify left))
     )
-    (property "Footprint" "" (id 2) (at 145.7452 80.01 0)
+    (property "Footprint" "Capacitor_SMD:C_0603_1608Metric" (id 2) (at 144.4752 80.01 0)
       (effects (font (size 1.27 1.27)) hide)
     )
-    (property "Datasheet" "~" (id 3) (at 144.78 76.2 0)
+    (property "Datasheet" "~" (id 3) (at 143.51 76.2 0)
       (effects (font (size 1.27 1.27)) hide)
     )
@@
   (symbol (lib_id "Device:R") (at 132.08 68.58 0)
     (in_bom yes) (on_board yes) (fields_autoplaced)
-    (property "Reference" "R?" (id 0) (at 133.858 67.6715 0)
+    (property "Reference" "R46" (id 0) (at 133.858 67.6715 0)
       (effects (font (size 1.27 1.27)) (justify left))
     )
@@
   (symbol (lib_id "power:GND") (at 132.08 82.55 0)
     (in_bom yes) (on_board yes) (fields_autoplaced)
-    (property "Reference" "#PWR?" (id 0) (at 132.08 88.9 0)
+    (property "Reference" "#PWR0202" (id 0) (at 132.08 88.9 0)
       (effects (font (size 1.27 1.27)) hide)
     )
@@
   (symbol (lib_id "Device:R") (at 123.19 81.28 0)
     (in_bom yes) (on_board yes) (fields_autoplaced)
-    (property "Reference" "R?" (id 0) (at 124.968 80.3715 0)
+    (property "Reference" "R45" (id 0) (at 124.968 80.3715 0)
       (effects (font (size 1.27 1.27)) (justify left))
     )
@@
     (pin "2")
   )
-  (symbol (lib_id "power:GND") (at 144.78 80.01 0)
+  (symbol (lib_id "power:GND") (at 143.51 80.01 0)
     (in_bom yes) (on_board yes) (fields_autoplaced)
-    (property "Reference" "#PWR?" (id 0) (at 144.78 86.36 0)
+    (property "Reference" "#PWR0203" (id 0) (at 143.51 86.36 0)
       (effects (font (size 1.27 1.27)) hide)
     )
-    (property "Value" "GND" (id 1) (at 144.78 84.5725 0))
-    (property "Footprint" "" (id 2) (at 144.78 80.01 0)
+    (property "Value" "GND" (id 1) (at 143.51 84.5725 0))
+    (property "Footprint" "" (id 2) (at 143.51 80.01 0)
       (effects (font (size 1.27 1.27)) hide)
     )
-    (property "Datasheet" "" (id 3) (at 144.78 80.01 0)
+    (property "Datasheet" "" (id 3) (at 143.51 80.01 0)
       (effects (font (size 1.27 1.27)) hide)
     )
@@
   (symbol (lib_id "Transistor_FET:2N7002") (at 129.54 77.47 0)
     (in_bom yes) (on_board yes) (fields_autoplaced)
-    (property "Reference" "Q?" (id 0) (at 134.747 76.5615 0)
+    (property "Reference" "Q14" (id 0) (at 134.747 76.5615 0)
       (effects (font (size 1.27 1.27)) (justify left))
     )
