File: alarm_panel_breakout/Sonoff_Relay_Output.kicad_sch (KiCad schematic)
At the start: 5 parts

Commit message: alarm panel initial layout
Parts:
- gave numbers to parts that had none: 5
Changed lines of the file:
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@@
   (symbol (lib_id "Device:R") (at 135.89 111.76 0)
     (in_bom yes) (on_board yes) (fields_autoplaced)
-    (property "Reference" "R?" (id 0) (at 137.668 110.8515 0)
+    (property "Reference" "R9" (id 0) (at 137.668 110.8515 0)
       (effects (font (size 1.27 1.27)) (justify left))
     )
@@
   (symbol (lib_id "Diode:1N4148") (at 144.78 91.44 270)
     (in_bom yes) (on_board yes) (fields_autoplaced)
-    (property "Reference" "D?" (id 0) (at 146.812 90.5315 90)
+    (property "Reference" "D2" (id 0) (at 146.812 90.5315 90)
       (effects (font (size 1.27 1.27)) (justify left))
     )
@@
   (symbol (lib_id "power:GND") (at 144.78 113.03 0)
     (in_bom yes) (on_board yes) (fields_autoplaced)
-    (property "Reference" "#PWR?" (id 0) (at 144.78 119.38 0)
+    (property "Reference" "#PWR0163" (id 0) (at 144.78 119.38 0)
       (effects (font (size 1.27 1.27)) hide)
     )
@@
   (symbol (lib_id "power:+5V") (at 152.4 85.09 0)
     (in_bom yes) (on_board yes) (fields_autoplaced)
-    (property "Reference" "#PWR?" (id 0) (at 152.4 88.9 0)
+    (property "Reference" "#PWR0162" (id 0) (at 152.4 88.9 0)
       (effects (font (size 1.27 1.27)) hide)
     )
@@
   (symbol (lib_id "Evan's misc parts:sonoff_relay") (at 166.37 92.71 0)
     (in_bom yes) (on_board yes) (fields_autoplaced)
-    (property "Reference" "K?" (id 0) (at 177.292 93.189 0)
+    (property "Reference" "K1" (id 0) (at 177.292 93.189 0)
       (effects (font (size 1.27 1.27)) (justify left))
     )
@@
   (symbol (lib_id "Device:R") (at 130.81 107.95 90)
     (in_bom yes) (on_board yes) (fields_autoplaced)
-    (property "Reference" "R?" (id 0) (at 130.81 102.9675 90))
+    (property "Reference" "R8" (id 0) (at 130.81 102.9675 90))
     (property "Value" "1K" (id 1) (at 130.81 105.7426 90))
     (property "Footprint" "Resistor_SMD:R_0603_1608Metric" (id 2) (at 130.81 109.728 90)
@@
   (symbol (lib_id "power:GND") (at 135.89 115.57 0)
     (in_bom yes) (on_board yes) (fields_autoplaced)
-    (property "Reference" "#PWR?" (id 0) (at 135.89 121.92 0)
+    (property "Reference" "#PWR0164" (id 0) (at 135.89 121.92 0)
       (effects (font (size 1.27 1.27)) hide)
     )
@@
   (symbol (lib_id "Transistor_FET:2N7002") (at 142.24 107.95 0)
     (in_bom yes) (on_board yes) (fields_autoplaced)
-    (property "Reference" "Q?" (id 0) (at 147.447 107.0415 0)
+    (property "Reference" "Q1" (id 0) (at 147.447 107.0415 0)
       (effects (font (size 1.27 1.27)) (justify left))
     )
