File: alarm_panel_breakout/alarm_panel_breakout.kicad_sch (KiCad schematic)
At the start: 21 parts

Commit message: alarm panel initial layout
Parts:
- added J10: 12v bus, Connector_Phoenix_MC:PhoenixContact_MC_1,5_13-G-3.5_1x13_P3.50mm_Horizontal, symbol Connector_Generic:Conn_01x13
- added J11: inputs, Connector_Phoenix_MC:PhoenixContact_MC_1,5_13-G-3.5_1x13_P3.50mm_Horizontal, symbol Connector_Generic:Conn_01x13
- added J12: 5v bus, Connector_Phoenix_MC:PhoenixContact_MC_1,5_13-G-3.5_1x13_P3.50mm_Horizontal, symbol Connector_Generic:Conn_01x13
- added J13: gnd bus, Connector_Phoenix_MC:PhoenixContact_MC_1,5_13-G-3.5_1x13_P3.50mm_Horizontal, symbol Connector_Generic:Conn_01x13
- added J4: Input Mains, Connector_Phoenix_MC:PhoenixContact_MC_1,5_3-G-3.81_1x03_P3.81mm_Horizontal, symbol Connector_Generic:Conn_01x03
- added J6: Relay 1, Connector_Phoenix_MC:PhoenixContact_MC_1,5_3-G-3.81_1x03_P3.81mm_Horizontal, symbol Connector_Generic:Conn_01x03
- added J7: Relay 2, Connector_Phoenix_MC:PhoenixContact_MC_1,5_3-G-3.81_1x03_P3.81mm_Horizontal, symbol Connector_Generic:Conn_01x03
- added J8: Relay 3, Connector_Phoenix_MC:PhoenixContact_MC_1,5_3-G-3.81_1x03_P3.81mm_Horizontal, symbol Connector_Generic:Conn_01x03
- added J9: Barrel_Jack_Switch, Connector_BarrelJack:BarrelJack_GCT_DCJ200-10-A_Horizontal, symbol Connector:Barrel_Jack_Switch
- U3: renamed from U?; footprint (none) -> Evan's misc parts:YAAJ_DCDC_StepDown_LM2596
- gave numbers to parts that had none: 20
Connections:
- net +12V: now also J10.1 (Pin_1), J10.10 (Pin_10), J10.11 (Pin_11), J10.12 (Pin_12), J10.13 (Pin_13), J10.2 (Pin_2), J10.3 (Pin_3), J10.4 (Pin_4), J10.5 (Pin_5), J10.6 (Pin_6), J10.7 (Pin_7), J10.8 (Pin_8), J10.9 (Pin_9), J9.1
- net +5V: now also J12.1 (Pin_1), J12.10 (Pin_10), J12.11 (Pin_11), J12.12 (Pin_12), J12.13 (Pin_13), J12.2 (Pin_2), J12.3 (Pin_3), J12.4 (Pin_4), J12.5 (Pin_5), J12.6 (Pin_6), J12.7 (Pin_7), J12.8 (Pin_8), J12.9 (Pin_9)
- net GND: now also J13.1 (Pin_1), J13.10 (Pin_10), J13.11 (Pin_11), J13.12 (Pin_12), J13.13 (Pin_13), J13.2 (Pin_2), J13.3 (Pin_3), J13.4 (Pin_4), J13.5 (Pin_5), J13.6 (Pin_6), J13.7 (Pin_7), J13.8 (Pin_8), J13.9 (Pin_9), J9.2, J9.3
- new net Earth: J4.3 (Pin_3)
- new net Hot: J4.1 (Pin_1)
- new net In_19: J11.11 (Pin_11)
- new net In_23: J11.10 (Pin_10)
- new net In_25: J11.7 (Pin_7)
- new net In_26: J11.8 (Pin_8)
- new net In_27: J11.9 (Pin_9)
- new net In_32: J11.5 (Pin_5)
- new net In_33: J11.6 (Pin_6)
- new net In_34: J11.3 (Pin_3)
- new net In_35: J11.4 (Pin_4)
- new net In_36: J11.1 (Pin_1)
- new net In_39: J11.2 (Pin_2)
- new net In_4: J11.13 (Pin_13)
- new net In_5: J11.12 (Pin_12)
- new net Neutral: J4.2 (Pin_2), J6.3 (Pin_3), J7.3 (Pin_3), J8.3 (Pin_3)
- new net Relay1: J6.1 (Pin_1)
- new net Relay1_2: J6.2 (Pin_2)
- new net Relay2: J7.1 (Pin_1)
- new net Relay2_2: J7.2 (Pin_2)
- new net Relay3: J8.1 (Pin_1)
- new net Relay3_2: J8.2 (Pin_2)
Other:
- moved on the sheet: U3
