File: alarm_panel_breakout/alarm_panel_breakout.kicad_pcb (KiCad board)
At the start: 2 copper layers, 99.7 x 99.7 mm, 114 parts, among them J1 Conn_02x05_Odd_Even, J10 12v bus, J11 inputs, J12 5v bus, J13 gnd bus, J2 Conn_02x03_Odd_Even, J3 bme280, J4 Input Mains, J6 Relay 1, J7 Relay 2, J8 Relay 3, J9 Barrel_Jack_Switch, K1 sonoff_relay, K2 sonoff_relay, K3 sonoff_relay, Q1 2N7002, Q10 2N7002, Q11 2N7002, Q12 2N7002, Q13 2N7002, Q14 2N7002, Q15 2N7002, Q16 2N7002, Q2 2N7002, Q3 2N7002, Q4 2N7002, Q5 2N7002, Q6 2N7002, Q7 2N7002, Q8 2N7002, Q9 2N7002, SW1 SW_MEC_5E, U1 ESP32-WROOM-32U, U2 LD1117S33TR_SOT223, U3 YAAJ_DCDC_StepDown_LM2596

Commit message: generated gerbers
Parts:
- added G***: LOGO, Evan's misc parts:OSHW gear, F.Cu at (89.6, 13.0)
- added G***: LOGO, Evan's misc parts:Evan Logo, F.Cu at (22.4, 64.4)
Routing:
- net GND: track 0.00 -> 3.04 mm
- net +3V3: track 254.2 -> 253.0 mm, vias 21 -> 20
- net /ESP_IO0: track 26.2 -> 25.1 mm
- net /ESP_IO32: track 29.2 -> 28.6 mm
- net /ESP_IO34: track 35.0 -> 34.5 mm
- net /ESP_EN: track 117.1 -> 116.7 mm, vias 3 -> 2
Other:
- board text added: "12"
- board text added: "12v"
- board text added: "13"
- board text added: "14"
- board text added: "15"
- board text added: "19"
- board text added: "21"
- board text added: "22"
- board text added: "23"
- board text added: "25"
- board text added: "26"
- board text added: "27"
- board text added: "2N7002"
- board text added: "32"
- board text added: "33"
- board text added: "34"
- board text added: "35"
- board text added: "36"
- board text added: "39"
- board text added: "3v3"
- board text added: "4"
- board text added: "5"
- board text added: "5v"
- board text added: "Buffered, protecred alarm panel board"
- board text added: "En"
- board text added: "IO 16"
- board text added: "IO 17"
- board text added: "IO 18"
- board text added: "IO0"
- board text added: "IO1"
- board text added: "IO3"
- board text added: "NO"
- board text added: "abzman2k.wordpress.com"
- board text added: "all pulled down by 10k"
- board text added: "earth"
- board text added: "gnd"
- board text added: "hot"
- board text added: "input mains"
- board text added: "neutral"
- board text added: "reset"
- board text added: "up to 60(?)v DC"
