File: Xc9572 breakout/Xc9572 breakout.kicad_pcb (KiCad board)
At the start: 2 copper layers, 50.8 x 43.2 mm, 49 parts, among them J1 programming header, J10 1-6, J11 1-8, J12 1-9/GCK1, J13 1-11/GCK2, J14 1-14/GCK3, J15 1-15, J16 1-17, J17 2-2, J18 2-5, J19 2-6, J2 Vcc INT, J20 2-8, J21 2-9/GSR, J22 2-11/GTS2, J23 2-14/GTS1, J24 2-15, J25 2-17, J26 3-2, J27 3-5, J28 3-8, J29 3-9, J3 Vcc IO, J30 3-11, J31 3-14, J32 3-15, J33 3-17, J34 4-2, J35 4-5, J36 4-8, J37 4-9, J38 4-11, J39 4-14, J4 power jumper, J40 4-15, J41 4-17, J5 5v, J7 Gnd, J8 1-2, J9 1-5, U1 XC9572-PLCC44

Commit message: generated gerbers
Parts:
- moved C2 0.28 mm to (91.4, 49.9)
- moved C1 0.27 mm to (98.0, 53.4)
Changed lines of the file:
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@@
       (layerselection 0x00010fc_ffffffff)
       (disableapertmacros false)
-      (usegerberextensions false)
+      (usegerberextensions true)
       (usegerberattributes true)
       (usegerberadvancedattributes true)
@@
       (plotinvisibletext false)
       (sketchpadsonfab false)
-      (subtractmaskfromsilk false)
+      (subtractmaskfromsilk true)
       (outputformat 1)
       (mirror false)
-      (drillshape 1)
+      (drillshape 0)
       (scaleselection 1)
-      (outputdirectory "")
+      (outputdirectory "Xc9572 breakout-gerbers")
     )
   )
@@
       (effects (font (size 1 1) (thickness 0.15)))
     )
-    (fp_text value "2-11/GTS2" (at 0 2.33) (layer "F.SilkS")
+    (fp_text value "2-11/GTS2" (at 4.7752 0.0254) (layer "F.SilkS")
       (effects (font (size 0.7 0.7) (thickness 0.1)))
     )
@@
   )
   (footprint "Capacitor_SMD:C_0603_1608Metric" (layer "F.Cu")
-    (at 91.44 50.165 -90)
+    (at 91.44 49.8856 -90)
     (descr "Capacitor SMD 0603 (1608 Metric), square (rectangular) end terminal, IPC_7351 nominal, (Body size source: IPC-SM-782 page 76, https://www.pcb-3d.com/wordpress/wp-content/uploads/ipc-sm-782a_amendment_1_and_2.pdf), generated with kicad-footprint-generator")
     (tags "capacitor")
@@
   )
   (footprint "Capacitor_SMD:C_0603_1608Metric" (layer "F.Cu")
-    (at 97.79 53.34 -90)
+    (at 98.044 53.4162 -90)
     (descr "Capacitor SMD 0603 (1608 Metric), square (rectangular) end terminal, IPC_7351 nominal, (Body size source: IPC-SM-782 page 76, https://www.pcb-3d.com/wordpress/wp-content/uploads/ipc-sm-782a_amendment_1_and_2.pdf), generated with kicad-footprint-generator")
     (tags "capacitor")
@@
       (effects (font (size 1 1) (thickness 0.15)))
     )
-    (fp_text value "Vcc INT" (at 0 2.33) (layer "F.SilkS")
+    (fp_text value "Vcc INT" (at -3.556 -0.0508) (layer "F.SilkS")
       (effects (font (size 0.7 0.7) (thickness 0.1)))
     )
@@
       (effects (font (size 1 1) (thickness 0.15)))
     )
-    (fp_text value "2-14/GTS1" (at 0 2.33) (layer "F.SilkS")
+    (fp_text value "2-14/GTS1" (at 0.4572 2.2606) (layer "F.SilkS")
       (effects (font (size 0.7 0.7) (thickness 0.1)))
     )
@@
     (effects (font (size 1 1) (thickness 0.15)) (justify mirror))
   )
-  (gr_text "Vcc IO" (at 95.37 48.235 90) (layer "F.SilkS")
+  (gr_text "Vcc IO" (at 95.7072 49.1998 90) (layer "F.SilkS")
     (effects (font (size 1 1) (thickness 0.15)))
   )
@@
     (effects (font (size 1 1) (thickness 0.15)))
   )
-  (gr_text "Vcc INT" (at 92.83 48.235 90) (layer "F.SilkS")
+  (gr_text "Vcc INT" (at 93.091 49.0474 90) (layer "F.SilkS")
     (effects (font (size 1 1) (thickness 0.15)))
   )
@@
   (segment (start 109.855 63.5) (end 113.665 63.5) (width 0.25) (layer "B.Cu") (net 3))
   (segment (start 92.83 51.95) (end 93.345 51.435) (width 0.25) (layer "F.Cu") (net 4))
-  (segment (start 91.44 49.53) (end 93.345 51.435) (width 0.25) (layer "F.Cu") (net 4))
+  (segment (start 93.345 51.435) (end 93.8403 50.9397) (width 0.25) (layer "F.Cu") (net 4))
   (segment (start 116.84 66.2825) (end 116.84 64.77) (width 0.25) (layer "F.Cu") (net 4))
+  (segment (start 91.44 49.1106) (end 92.0112 49.1106) (width 0.25) (layer "F.Cu") (net 4))
   (segment (start 124.46 50.5575) (end 124.46 52.705) (width 0.25) (layer "F.Cu") (net 4))
   (segment (start 116.84 64.77) (end 117.475 64.135) (width 0.25) (layer "F.Cu") (net 4))
-  (segment (start 91.44 49.39) (end 91.44 49.53) (width 0.25) (layer "F.Cu") (net 4))
-  (segment (start 93.345 51.435) (end 104.14 40.64) (width 0.25) (layer "F.Cu") (net 4))
   (segment (start 92.83 53.315) (end 92.83 51.95) (width 0.25) (layer "F.Cu") (net 4))
+  (segment (start 93.8403 50.9397) (end 104.14 40.64) (width 0.25) (layer "F.Cu") (net 4))
+  (segment (start 92.0112 49.1106) (end 93.8403 50.9397) (width 0.25) (layer "F.Cu") (net 4))
   (via (at 124.46 52.705) (size 0.8) (drill 0.4) (layers "F.Cu" "B.Cu") (net 4))
   (via (at 117.475 64.135) (size 0.8) (drill 0.4) (layers "F.Cu" "B.Cu") (net 4))
@@
   (segment (start 96.765489 59.785489) (end 111.855489 59.785489) (width 0.25) (layer "B.Cu") (net 9))
   (segment (start 127.2425 60.96) (end 125.095 60.96) (width 0.25) (layer "F.Cu") (net 10))
-  (segment (start 97.79 52.565) (end 97.04 53.315) (width 0.25) (layer "F.Cu") (net 10))
+  (segment (start 97.7138 52.6412) (end 97.04 53.315) (width 0.25) (layer "F.Cu") (net 10))
   (segment (start 95.37 53.315) (end 100.425 48.26) (width 0.25) (layer "F.Cu") (net 10))
   (segment (start 97.04 53.315) (end 95.37 53.315) (width 0.25) (layer "F.Cu") (net 10))
   (segment (start 100.425 48.26) (end 101.6 48.26) (width 0.25) (layer "F.Cu") (net 10))
+  (segment (start 98.044 52.6412) (end 97.7138 52.6412) (width 0.25) (layer "F.Cu") (net 10))
   (via (at 125.095 60.96) (size 0.8) (drill 0.4) (layers "F.Cu" "B.Cu") (net 10))
   (segment (start 121.285 48.26) (end 101.6 48.26) (width 0.25) (layer "B.Cu") (net 10))
