File: Xc9572 breakout/Xc9572 breakout.kicad_sch (KiCad schematic)
At the start: 43 parts, among them J1 programming header, J10 1-6, J11 1-8, J12 1-9/GCK1, J13 1-11/GCK2, J14 1-14/GCK3, J15 1-15, J16 1-17, J17 2-2, J18 2-5, J19 2-6, J2 Vcc INT, J20 2-8, J21 2-9/GSR, J22 2-11/GTS2, J23 2-14/GTS1, J24 2-15, J25 2-17, J26 3-2, J27 3-5, J28 3-8, J29 3-9, J3 Vcc IO, J30 3-11, J31 3-14, J32 3-15, J33 3-17, J34 4-2, J35 4-5, J36 4-8, J37 4-9, J38 4-11, J39 4-14, J4 power jumper, J40 4-15, J41 4-17, J5 5v, J7 Gnd, J8 1-2, J9 1-5, U1 XC9572-PLCC44

Commit message: added gerbers, fixed ERC/DRC
Other:
- moved on the sheet: J5, J7
Changed lines of the file:
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@@
     (pin "1")
   )
-  (symbol (lib_id "Connector_Generic:Conn_01x01") (at 193.04 31.75 0) (unit 1)
-    (in_bom yes) (on_board yes)
-    (property "Reference" "J7" (id 0) (at 195.072 30.8415 0)
-      (effects (font (size 1.27 1.27)) (justify left))
-    )
-    (property "Value" "Gnd" (id 1) (at 197.485 31.75 0)
-      (effects (font (size 1.27 1.27)) (justify left))
-    )
-    (property "Footprint" "Connector_PinHeader_2.54mm:PinHeader_1x01_P2.54mm_Vertical" (id 2) (at 193.04 31.75 0)
-      (effects (font (size 1.27 1.27)) hide)
-    )
-    (property "Datasheet" "~" (id 3) (at 193.04 31.75 0)
+  (symbol (lib_id "Connector_Generic:Conn_01x01") (at 63.5 32.385 0) (unit 1)
+    (in_bom yes) (on_board yes)
+    (property "Reference" "J7" (id 0) (at 65.532 31.4765 0)
+      (effects (font (size 1.27 1.27)) (justify left))
+    )
+    (property "Value" "Gnd" (id 1) (at 67.945 32.385 0)
+      (effects (font (size 1.27 1.27)) (justify left))
+    )
+    (property "Footprint" "Connector_PinHeader_2.54mm:PinHeader_1x01_P2.54mm_Vertical" (id 2) (at 63.5 32.385 0)
+      (effects (font (size 1.27 1.27)) hide)
+    )
+    (property "Datasheet" "~" (id 3) (at 63.5 32.385 0)
       (effects (font (size 1.27 1.27)) hide)
     )
@@
     (pin "1")
   )
-  (symbol (lib_id "Connector_Generic:Conn_01x01") (at 193.04 25.4 0) (unit 1)
-    (in_bom yes) (on_board yes)
-    (property "Reference" "J5" (id 0) (at 195.072 24.4915 0)
-      (effects (font (size 1.27 1.27)) (justify left))
-    )
-    (property "Value" "5v" (id 1) (at 197.485 25.4 0)
-      (effects (font (size 1.27 1.27)) (justify left))
-    )
-    (property "Footprint" "Connector_PinHeader_2.54mm:PinHeader_1x01_P2.54mm_Vertical" (id 2) (at 193.04 25.4 0)
-      (effects (font (size 1.27 1.27)) hide)
-    )
-    (property "Datasheet" "~" (id 3) (at 193.04 25.4 0)
+  (symbol (lib_id "Connector_Generic:Conn_01x01") (at 63.5 26.035 0) (unit 1)
+    (in_bom yes) (on_board yes)
+    (property "Reference" "J5" (id 0) (at 65.532 25.1265 0)
+      (effects (font (size 1.27 1.27)) (justify left))
+    )
+    (property "Value" "5v" (id 1) (at 67.945 26.035 0)
+      (effects (font (size 1.27 1.27)) (justify left))
+    )
+    (property "Footprint" "Connector_PinHeader_2.54mm:PinHeader_1x01_P2.54mm_Vertical" (id 2) (at 63.5 26.035 0)
+      (effects (font (size 1.27 1.27)) hide)
+    )
+    (property "Datasheet" "~" (id 3) (at 63.5 26.035 0)
       (effects (font (size 1.27 1.27)) hide)
     )
@@
     (pin "2")
   )
-  (symbol (lib_id "power:GND") (at 187.96 31.75 0) (unit 1)
-    (in_bom yes) (on_board yes) (fields_autoplaced)
-    (property "Reference" "#PWR08" (id 0) (at 187.96 38.1 0)
-      (effects (font (size 1.27 1.27)) hide)
-    )
-    (property "Value" "GND" (id 1) (at 187.96 36.3125 0))
-    (property "Footprint" "" (id 2) (at 187.96 31.75 0)
-      (effects (font (size 1.27 1.27)) hide)
-    )
-    (property "Datasheet" "" (id 3) (at 187.96 31.75 0)
+  (symbol (lib_id "power:GND") (at 58.42 32.385 0) (unit 1)
+    (in_bom yes) (on_board yes) (fields_autoplaced)
+    (property "Reference" "#PWR08" (id 0) (at 58.42 38.735 0)
+      (effects (font (size 1.27 1.27)) hide)
+    )
+    (property "Value" "GND" (id 1) (at 58.42 36.9475 0))
+    (property "Footprint" "" (id 2) (at 58.42 32.385 0)
+      (effects (font (size 1.27 1.27)) hide)
+    )
+    (property "Datasheet" "" (id 3) (at 58.42 32.385 0)
       (effects (font (size 1.27 1.27)) hide)
     )
@@
     (pin "1")
   )
-  (symbol (lib_id "power:+5V") (at 187.96 25.4 0) (unit 1)
-    (in_bom yes) (on_board yes) (fields_autoplaced)
-    (property "Reference" "#PWR07" (id 0) (at 187.96 29.21 0)
-      (effects (font (size 1.27 1.27)) hide)
-    )
-    (property "Value" "+5V" (id 1) (at 187.96 21.7955 0))
-    (property "Footprint" "" (id 2) (at 187.96 25.4 0)
-      (effects (font (size 1.27 1.27)) hide)
-    )
-    (property "Datasheet" "" (id 3) (at 187.96 25.4 0)
-      (effects (font (size 1.27 1.27)) hide)
-    )
+  (symbol (lib_id "power:+5V") (at 58.42 26.035 0) (unit 1)
+    (in_bom yes) (on_board yes) (fields_autoplaced)
+    (property "Reference" "#PWR07" (id 0) (at 58.42 29.845 0)
+      (effects (font (size 1.27 1.27)) hide)
+    )
+    (property "Value" "+5V" (id 1) (at 58.42 22.4305 0))
+    (property "Footprint" "" (id 2) (at 58.42 26.035 0)
+      (effects (font (size 1.27 1.27)) hide)
+    )
+    (property "Datasheet" "" (id 3) (at 58.42 26.035 0)
+      (effects (font (size 1.27 1.27)) hide)
+    )
