File: dual LED board/dual LED board.kicad_pcb (KiCad board)
At the start: 2 copper layers, 23.6 x 20.3 mm, 28 parts, among them J1 Conn_01x02, J2 Conn_01x08

Commit message: generated gerbers
Changed lines of the file:
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@@
       (layerselection 0x00010fc_ffffffff)
       (disableapertmacros false)
-      (usegerberextensions false)
+      (usegerberextensions true)
       (usegerberattributes true)
       (usegerberadvancedattributes true)
@@
       (plotinvisibletext false)
       (sketchpadsonfab false)
-      (subtractmaskfromsilk false)
+      (subtractmaskfromsilk true)
       (outputformat 1)
       (mirror false)
-      (drillshape 1)
+      (drillshape 0)
       (scaleselection 1)
-      (outputdirectory "")
+      (outputdirectory "dual LED board-gerbers")
     )
   )
@@
   (segment (start 163.422 58.457) (end 170.05 58.457) (width 0.25) (layer "F.Cu") (net 1))
   (segment (start 172.85 67.186) (end 171.45 65.786) (width 0.25) (layer "F.Cu") (net 2))
-  (segment (start 170.561 75.819) (end 170.688 75.946) (width 0.25) (layer "F.Cu") (net 2))
   (segment (start 172.85 61.344) (end 172.72 61.214) (width 0.25) (layer "F.Cu") (net 2))
   (segment (start 172.85 72.935) (end 172.85 72.52) (width 0.25) (layer "F.Cu") (net 2))
