File: simple_button_breakout/simple_button_breakout.kicad_pcb (KiCad board)
At the start: 2 copper layers, 75.3 x 60.3 mm, 87 parts, among them J1 Conn_02x05_Odd_Even, J10 Conn_01x03, J11 Conn_01x03, J12 Conn_01x03, J13 Conn_01x03, J14 Conn_01x03, J15 Conn_01x03, J16 UJ2-MIBH-G-SMT-TR, J2 bme280, J3 Conn_02x03_Odd_Even, J4 Conn_01x03, J5 Conn_01x03, J6 Conn_01x03, J7 Conn_01x03, J8 Conn_01x03, J9 Conn_01x03, SW1 SW_MEC_5E, U1 ESP32-WROOM-32U, U2 LD1117S33TR_SOT223

Commit message: generated gerbers
Other:
- board text added: "12"
- board text added: "13"
- board text added: "14"
- board text added: "15"
- board text added: "16"
- board text added: "17"
- board text added: "18"
- board text added: "19"
- board text added: "23"
- board text added: "25"
- board text added: "26"
- board text added: "27"
- board text added: "32"
- board text added: "33"
- board text added: "4"
- board text added: "5"
- board text added: "5v"
- board text added: "En"
- board text added: "IO0"
- board text added: "IO1"
- board text added: "IO3"
- board text added: "gnd"
