File: rp2040 rs485 scale breakout/nau7802module.kicad_sch (KiCad schematic)
At the start: 17 parts, among them J15 channel 1, J16 channel 2, J17 cap, J18 i2c pullips, U4 NAU7802SGI

Commit message: motor driver and scale pcb gerbers
Parts:
- renumbered C12 to C17, C13 to C18, C14 to C19, C15 to C20, C16 to C21, C22 to C23, J15 to J19, J16 to J20, J17 to J21, J18 to J22, R29 to R33, R30 to R34, R31 to R35, R32 to R36, R37 to R39, R38 to R40, U4 to U5
Changed lines of the file:
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@@
   (symbol (lib_id "Device:R") (at 76.2 59.055 90) (mirror x)
     (in_bom yes) (on_board yes)
-    (property "Reference" "R37" (id 0) (at 76.2 54.0725 90))
+    (property "Reference" "R39" (id 0) (at 76.2 54.0725 90))
     (property "Value" "47" (id 1) (at 76.2 56.8476 90))
     (property "Footprint" "Resistor_SMD:R_0603_1608Metric" (id 2) (at 76.2 57.277 90)
@@
   (symbol (lib_id "Connector_Generic:Conn_01x04") (at 49.53 70.485 180)
     (in_bom yes) (on_board yes)
-    (property "Reference" "J16" (id 0) (at 49.53 60.1685 0))
+    (property "Reference" "J20" (id 0) (at 49.53 60.1685 0))
     (property "Value" "channel 2" (id 1) (at 46.99 62.865 0))
     (property "Footprint" "Connector_JST:JST_XH_B4B-XH-A_1x04_P2.50mm_Vertical" (id 2) (at 49.53 70.485 0)
@@
   (symbol (lib_id "Device:R") (at 95.25 48.895 90) (mirror x)
     (in_bom yes) (on_board yes) (fields_autoplaced)
-    (property "Reference" "R29" (id 0) (at 95.25 43.9125 90))
+    (property "Reference" "R33" (id 0) (at 95.25 43.9125 90))
     (property "Value" "47" (id 1) (at 95.25 46.6876 90))
     (property "Footprint" "Resistor_SMD:R_0603_1608Metric" (id 2) (at 95.25 47.117 90)
@@
   (symbol (lib_id "Device:C") (at 81.915 66.04 0)
     (in_bom yes) (on_board yes)
-    (property "Reference" "C22" (id 0) (at 76.835 64.135 0)
+    (property "Reference" "C23" (id 0) (at 76.835 64.135 0)
       (effects (font (size 1.27 1.27)) (justify left))
     )
@@
   (symbol (lib_id "Device:C") (at 147.32 34.925 0)
     (in_bom yes) (on_board yes) (fields_autoplaced)
-    (property "Reference" "C16" (id 0) (at 150.241 34.0165 0)
+    (property "Reference" "C21" (id 0) (at 150.241 34.0165 0)
       (effects (font (size 1.27 1.27)) (justify left))
     )
@@
   (symbol (lib_id "Connector_Generic:Conn_01x04") (at 49.53 53.34 180)
     (in_bom yes) (on_board yes)
-    (property "Reference" "J15" (id 0) (at 49.53 43.0235 0))
+    (property "Reference" "J19" (id 0) (at 49.53 43.0235 0))
     (property "Value" "channel 1" (id 1) (at 46.355 45.72 0))
     (property "Footprint" "Connector_JST:JST_XH_B4B-XH-A_1x04_P2.50mm_Vertical" (id 2) (at 49.53 53.34 0)
@@
   (symbol (lib_id "Device:R") (at 193.675 50.8 0) (mirror y)
     (in_bom yes) (on_board yes) (fields_autoplaced)
-    (property "Reference" "R32" (id 0) (at 191.897 49.8915 0)
+    (property "Reference" "R36" (id 0) (at 191.897 49.8915 0)
       (effects (font (size 1.27 1.27)) (justify left))
     )
@@
   (symbol (lib_id "Device:C") (at 102.87 52.705 0)
     (in_bom yes) (on_board yes) (fields_autoplaced)
-    (property "Reference" "C13" (id 0) (at 105.791 51.7965 0)
+    (property "Reference" "C18" (id 0) (at 105.791 51.7965 0)
       (effects (font (size 1.27 1.27)) (justify left))
     )
@@
   (symbol (lib_id "Device:R") (at 76.2 74.295 90) (mirror x)
     (in_bom yes) (on_board yes)
-    (property "Reference" "R38" (id 0) (at 76.2 69.3125 90))
+    (property "Reference" "R40" (id 0) (at 76.2 69.3125 90))
     (property "Value" "47" (id 1) (at 76.2 72.0876 90))
     (property "Footprint" "Resistor_SMD:R_0603_1608Metric" (id 2) (at 76.2 72.517 90)
@@
   (symbol (lib_id "Device:R") (at 185.42 50.8 0) (mirror y)
     (in_bom yes) (on_board yes) (fields_autoplaced)
-    (property "Reference" "R31" (id 0) (at 183.642 49.8915 0)
+    (property "Reference" "R35" (id 0) (at 183.642 49.8915 0)
       (effects (font (size 1.27 1.27)) (justify left))
     )
@@
   (symbol (lib_id "Connector_Generic:Conn_01x02") (at 90.805 66.675 180)
     (in_bom yes) (on_board yes)
-    (property "Reference" "J17" (id 0) (at 86.995 65.405 0))
+    (property "Reference" "J21" (id 0) (at 86.995 65.405 0))
     (property "Value" "cap" (id 1) (at 86.995 67.31 0))
     (property "Footprint" "Jumper:SolderJumper-2_P1.3mm_Bridged_RoundedPad1.0x1.5mm" (id 2) (at 90.805 66.675 0)
@@
   (symbol (lib_id "Device:C") (at 135.89 34.925 0)
     (in_bom yes) (on_board yes) (fields_autoplaced)
-    (property "Reference" "C15" (id 0) (at 138.811 34.0165 0)
+    (property "Reference" "C20" (id 0) (at 138.811 34.0165 0)
       (effects (font (size 1.27 1.27)) (justify left))
     )
@@
   (symbol (lib_id "Device:R") (at 95.25 56.515 90) (mirror x)
     (in_bom yes) (on_board yes) (fields_autoplaced)
-    (property "Reference" "R30" (id 0) (at 95.25 51.5325 90))
+    (property "Reference" "R34" (id 0) (at 95.25 51.5325 90))
     (property "Value" "47" (id 1) (at 95.25 54.3076 90))
     (property "Footprint" "Resistor_SMD:R_0603_1608Metric" (id 2) (at 95.25 54.737 90)
@@
   (symbol (lib_id "Evan's misc parts:NAU7802SGI") (at 120.65 51.435 0)
     (in_bom yes) (on_board yes) (fields_autoplaced)
-    (property "Reference" "U4" (id 0) (at 146.05 41.8876 0)
+    (property "Reference" "U5" (id 0) (at 146.05 41.8876 0)
       (effects (font (size 1.524 1.524)))
     )
@@
   (symbol (lib_id "Device:C") (at 109.22 68.58 0)
     (in_bom yes) (on_board yes) (fields_autoplaced)
-    (property "Reference" "C14" (id 0) (at 112.141 67.6715 0)
+    (property "Reference" "C19" (id 0) (at 112.141 67.6715 0)
       (effects (font (size 1.27 1.27)) (justify left))
     )
@@
   (symbol (lib_id "Connector_Generic:Conn_01x03") (at 189.865 42.545 90) (mirror x)
     (in_bom yes) (on_board yes) (fields_autoplaced)
-    (property "Reference" "J18" (id 0) (at 185.293 41.6365 90)
+    (property "Reference" "J22" (id 0) (at 185.293 41.6365 90)
       (effects (font (size 1.27 1.27)) (justify left))
     )
@@
   (symbol (lib_id "Device:C") (at 95.885 70.485 0)
     (in_bom yes) (on_board yes) (fields_autoplaced)
-    (property "Reference" "C12" (id 0) (at 98.806 69.5765 0)
-      (effects (font (size 1.27 1.27)) (justify left))
-    )
+    (property "Reference" "C17" (id 0) (at 98.806 69.5765 0)
+      (effects (font (size 1.27 1.27)) (justify left))
+    )
