File: cord reel detent ring/cord reel detent ring.kicad_pcb (KiCad board)
At the start: 2 copper layers, 33.3 x 27.1 mm, 6 parts, among them J1 Conn_01x01, J2 Conn_01x01, J3 Conn_01x01, J4 Conn_01x01

Commit message: lots of stuff, I don't even know
Parts:
- added G***: LOGO, Evan's parts:pcbway logo, B.Cu at (-0.64, -7.62)
- added J5: Conn_01x01, Connector_PinHeader_2.54mm:PinHeader_1x01_P2.54mm_Vertical, F.Cu at (-3.17, 6.99)
- moved G*** 16.1 mm to (0.64, 6.99)
- moved J2 3.89 mm to (3.81, -12.1)
- moved J3 3.67 mm to (-3.17, -12.1)
