File: cord reel detent ring/cord reel detent ring.kicad_sch (KiCad schematic)
At the start: 4 parts, among them J1 Conn_01x01, J2 Conn_01x01, J3 Conn_01x01, J4 Conn_01x01

Commit message: lots of stuff, I don't even know
Parts:
- added J5: Conn_01x01, Connector_PinHeader_2.54mm:PinHeader_1x01_P2.54mm_Vertical, symbol Connector_Generic:Conn_01x01
Connections:
- net at J1.1 (Pin_1), J2.1 (Pin_1), J3.1 (Pin_1)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: now also J5.1 (Pin_1)
Changed lines of the file:
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@@
-(kicad_sch (version 20211123) (generator eeschema)
+(kicad_sch (version 20230121) (generator eeschema)
   (paper "A4")
   (junction (at 88.9 84.455) (diameter 0) (color 0 0 0 0)
+  )
+  (junction (at 88.9 95.25) (diameter 0) (color 0 0 0 0)
   )
   (junction (at 88.9 74.295) (diameter 0) (color 0 0 0 0)
   )
   (wire (pts (xy 90.805 84.455) (xy 88.9 84.455))
-    (stroke (width 0) (type default) (color 0 0 0 0))
+    (stroke (width 0) (type default))
   )
   (wire (pts (xy 88.9 74.295) (xy 88.9 64.77))
-    (stroke (width 0) (type default) (color 0 0 0 0))
+    (stroke (width 0) (type default))
   )
   (wire (pts (xy 90.805 95.25) (xy 88.9 95.25))
-    (stroke (width 0) (type default) (color 0 0 0 0))
+    (stroke (width 0) (type default))
   )
   (wire (pts (xy 88.9 84.455) (xy 88.9 74.295))
-    (stroke (width 0) (type default) (color 0 0 0 0))
+    (stroke (width 0) (type default))
   )
   (wire (pts (xy 88.9 95.25) (xy 88.9 84.455))
-    (stroke (width 0) (type default) (color 0 0 0 0))
+    (stroke (width 0) (type default))
   )
   (wire (pts (xy 90.17 74.295) (xy 88.9 74.295))
-    (stroke (width 0) (type default) (color 0 0 0 0))
+    (stroke (width 0) (type default))
   )
-  (symbol (lib_id "Connector_Generic:Conn_01x01") (at 95.25 74.295 0) (unit 1)
-    (in_bom yes) (on_board yes) (fields_autoplaced)
-    (property "Reference" "J2" (id 0) (at 97.282 73.3865 0)
+  (wire (pts (xy 88.9 106.045) (xy 88.9 95.25))
+    (stroke (width 0) (type default))
+  )
+  (wire (pts (xy 90.805 106.045) (xy 88.9 106.045))
+    (stroke (width 0) (type default))
+  )
+  (symbol (lib_id "Connector_Generic:Conn_01x01") (at 95.885 106.045 0) (unit 1)
+    (in_bom yes) (on_board yes) (dnp no) (fields_autoplaced)
+    (property "Reference" "J5" (at 97.917 105.1365 0)
       (effects (font (size 1.27 1.27)) (justify left))
     )
-    (property "Value" "Conn_01x01" (id 1) (at 97.282 76.1616 0)
+    (property "Value" "Conn_01x01" (at 97.917 107.9116 0)
       (effects (font (size 1.27 1.27)) (justify left))
     )
-    (property "Footprint" "Connector_PinHeader_2.54mm:PinHeader_1x01_P2.54mm_Vertical" (id 2) (at 95.25 74.295 0)
+    (property "Footprint" "Connector_PinHeader_2.54mm:PinHeader_1x01_P2.54mm_Vertical" (at 95.885 106.045 0)
       (effects (font (size 1.27 1.27)) hide)
     )
-    (property "Datasheet" "~" (id 3) (at 95.25 74.295 0)
+    (property "Datasheet" "~" (at 95.885 106.045 0)
       (effects (font (size 1.27 1.27)) hide)
     )
     (pin "1")
+    (instances
+      (project "cord reel detent ring"
+        (path "/e63e39d7-6ac0-4ffd-8aa3-1841a4541b55"
+          (reference "J5") (unit 1)
+        )
+      )
+    )
   )
-  (symbol (lib_id "Connector_Generic:Conn_01x01") (at 93.98 64.77 0) (unit 1)
-    (in_bom yes) (on_board yes) (fields_autoplaced)
-    (property "Reference" "J1" (id 0) (at 96.012 63.8615 0)
+  (symbol (lib_id "Connector_Generic:Conn_01x01") (at 95.25 74.295 0) (unit 1)
+    (in_bom yes) (on_board yes) (dnp no) (fields_autoplaced)
+    (property "Reference" "J2" (at 97.282 73.3865 0)
       (effects (font (size 1.27 1.27)) (justify left))
     )
-    (property "Value" "Conn_01x01" (id 1) (at 96.012 66.6366 0)
+    (property "Value" "Conn_01x01" (at 97.282 76.1616 0)
       (effects (font (size 1.27 1.27)) (justify left))
     )
-    (property "Footprint" "Connector_PinHeader_2.54mm:PinHeader_1x01_P2.54mm_Vertical" (id 2) (at 93.98 64.77 0)
+    (property "Footprint" "Connector_PinHeader_2.54mm:PinHeader_1x01_P2.54mm_Vertical" (at 95.25 74.295 0)
       (effects (font (size 1.27 1.27)) hide)
     )
-    (property "Datasheet" "~" (id 3) (at 93.98 64.77 0)
+    (property "Datasheet" "~" (at 95.25 74.295 0)
       (effects (font (size 1.27 1.27)) hide)
     )
     (pin "1")
+    (instances
+      (project "cord reel detent ring"
+        (path "/e63e39d7-6ac0-4ffd-8aa3-1841a4541b55"
+          (reference "J2") (unit 1)
+        )
+      )
+    )
   )
-  (symbol (lib_id "Connector_Generic:Conn_01x01") (at 95.885 95.25 0) (unit 1)
-    (in_bom yes) (on_board yes) (fields_autoplaced)
-    (property "Reference" "J4" (id 0) (at 97.917 94.3415 0)
+  (symbol (lib_id "Connector_Generic:Conn_01x01") (at 93.98 64.77 0) (unit 1)
+    (in_bom yes) (on_board yes) (dnp no) (fields_autoplaced)
+    (property "Reference" "J1" (at 96.012 63.8615 0)
       (effects (font (size 1.27 1.27)) (justify left))
     )
-    (property "Value" "Conn_01x01" (id 1) (at 97.917 97.1166 0)
+    (property "Value" "Conn_01x01" (at 96.012 66.6366 0)
       (effects (font (size 1.27 1.27)) (justify left))
     )
-    (property "Footprint" "Connector_PinHeader_2.54mm:PinHeader_1x01_P2.54mm_Vertical" (id 2) (at 95.885 95.25 0)
+    (property "Footprint" "Connector_PinHeader_2.54mm:PinHeader_1x01_P2.54mm_Vertical" (at 93.98 64.77 0)
       (effects (font (size 1.27 1.27)) hide)
     )
-    (property "Datasheet" "~" (id 3) (at 95.885 95.25 0)
+    (property "Datasheet" "~" (at 93.98 64.77 0)
       (effects (font (size 1.27 1.27)) hide)
     )
     (pin "1")
+    (instances
+      (project "cord reel detent ring"
+        (path "/e63e39d7-6ac0-4ffd-8aa3-1841a4541b55"
+          (reference "J1") (unit 1)
+        )
+      )
+    )
   )
-  (symbol (lib_id "Connector_Generic:Conn_01x01") (at 95.885 84.455 0) (unit 1)
-    (in_bom yes) (on_board yes) (fields_autoplaced)
-    (property "Reference" "J3" (id 0) (at 97.917 83.5465 0)
+  (symbol (lib_id "Connector_Generic:Conn_01x01") (at 95.885 95.25 0) (unit 1)
+    (in_bom yes) (on_board yes) (dnp no) (fields_autoplaced)
+    (property "Reference" "J4" (at 97.917 94.3415 0)
       (effects (font (size 1.27 1.27)) (justify left))
     )
-    (property "Value" "Conn_01x01" (id 1) (at 97.917 86.3216 0)
+    (property "Value" "Conn_01x01" (at 97.917 97.1166 0)
       (effects (font (size 1.27 1.27)) (justify left))
     )
-    (property "Footprint" "Connector_PinHeader_2.54mm:PinHeader_1x01_P2.54mm_Vertical" (id 2) (at 95.885 84.455 0)
+    (property "Footprint" "Connector_PinHeader_2.54mm:PinHeader_1x01_P2.54mm_Vertical" (at 95.885 95.25 0)
       (effects (font (size 1.27 1.27)) hide)
     )
-    (property "Datasheet" "~" (id 3) (at 95.885 84.455 0)
+    (property "Datasheet" "~" (at 95.885 95.25 0)
       (effects (font (size 1.27 1.27)) hide)
     )
     (pin "1")
+    (instances
+      (project "cord reel detent ring"
+        (path "/e63e39d7-6ac0-4ffd-8aa3-1841a4541b55"
+          (reference "J4") (unit 1)
+        )
+      )
+    )
+  )
+  (symbol (lib_id "Connector_Generic:Conn_01x01") (at 95.885 84.455 0) (unit 1)
+    (in_bom yes) (on_board yes) (dnp no) (fields_autoplaced)
+    (property "Reference" "J3" (at 97.917 83.5465 0)
+      (effects (font (size 1.27 1.27)) (justify left))
+    )
+    (property "Value" "Conn_01x01" (at 97.917 86.3216 0)
+      (effects (font (size 1.27 1.27)) (justify left))
+    )
+    (property "Footprint" "Connector_PinHeader_2.54mm:PinHeader_1x01_P2.54mm_Vertical" (at 95.885 84.455 0)
+      (effects (font (size 1.27 1.27)) hide)
+    )
+    (property "Datasheet" "~" (at 95.885 84.455 0)
+      (effects (font (size 1.27 1.27)) hide)
+    )
+    (pin "1")
+    (instances
+      (project "cord reel detent ring"
+        (path "/e63e39d7-6ac0-4ffd-8aa3-1841a4541b55"
+          (reference "J3") (unit 1)
+        )
+      )
+    )
   )
   (sheet_instances
     (path "/" (page "1"))
   )
-  (symbol_instances
-    (path "/aa288a22-ea1d-474d-8dae-efe971580843"
-      (reference "J1") (unit 1) (value "Conn_01x01") (footprint "Connector_PinHeader_2.54mm:PinHeader_1x01_P2.54mm_Vertical")
-    )
-    (path "/3972d90f-ee24-4cf5-8d82-ff4abccf2f2b"
-      (reference "J2") (unit 1) (value "Conn_01x01") (footprint "Connector_PinHeader_2.54mm:PinHeader_1x01_P2.54mm_Vertical")
-    )
-    (path "/f37f4fd2-2740-4984-ac7f-f80065bd2757"
-      (reference "J3") (unit 1) (value "Conn_01x01") (footprint "Connector_PinHeader_2.54mm:PinHeader_1x01_P2.54mm_Vertical")
-    )
-    (path "/ad2c8427-faf3-46bd-a366-df5ea0d688b4"
-      (reference "J4") (unit 1) (value "Conn_01x01") (footprint "Connector_PinHeader_2.54mm:PinHeader_1x01_P2.54mm_Vertical")
-    )
-  )
 )
