File: i2c 24vout/i2c 24vout.kicad_pcb (KiCad board)
At the start: 2 copper layers, 123.2 x 50.2 mm, 82 parts, among them J1 power in, J10 Conn_01x01, J2 Conn_01x04, J3 Conn_01x04, J4 Conn_01x04, J5 Conn_01x04, J6 to qwiic breakout, J7 qwiic 1, J8 qwiic 2, J9 Conn_01x01, U1 ILQ620GB-X009, U2 ILQ620GB-X009, U3 ILQ620GB-X009, U4 ILQ620GB-X009, U5 PCA9685PW

Commit message: lots of stuff, I don't even know
Parts:
- added R40: 0, Resistor_SMD:R_0603_1608Metric, F.Cu at (106.9, 118.6)
- added R41: 0, Resistor_SMD:R_0603_1608Metric, F.Cu at (111.9, 118.6)
- added R42: 0, Resistor_SMD:R_0603_1608Metric, F.Cu at (116.8, 118.6)
- added R43: 0, Resistor_SMD:R_0603_1608Metric, F.Cu at (121.8, 118.6)
- added R44: 0, Resistor_SMD:R_0603_1608Metric, F.Cu at (129.5, 118.5)
- added R45: 0, Resistor_SMD:R_0603_1608Metric, F.Cu at (134.5, 118.5)
- added R46: 0, Resistor_SMD:R_0603_1608Metric, F.Cu at (139.4, 118.5)
- added R47: 0, Resistor_SMD:R_0603_1608Metric, F.Cu at (144.5, 118.5)
- added R48: 0, Resistor_SMD:R_0603_1608Metric, F.Cu at (152.1, 118.6)
- added R49: 0, Resistor_SMD:R_0603_1608Metric, F.Cu at (157.2, 118.6)
- added R50: 0, Resistor_SMD:R_0603_1608Metric, F.Cu at (162.2, 118.6)
- added R51: 0, Resistor_SMD:R_0603_1608Metric, F.Cu at (167.3, 118.6)
- added R52: 0, Resistor_SMD:R_0603_1608Metric, F.Cu at (174.8, 118.6)
- added R53: 0, Resistor_SMD:R_0603_1608Metric, F.Cu at (179.8, 118.6)
- added R54: 0, Resistor_SMD:R_0603_1608Metric, F.Cu at (184.8, 118.6)
- added R55: 0, Resistor_SMD:R_0603_1608Metric, F.Cu at (189.9, 118.6)
- moved U2 1.64 mm to (138.8, 111.8)
- moved R2 1.64 mm to (113.5, 105.1)
- moved R4 1.64 mm to (123.6, 105.1)
- moved U1 1.64 mm to (116.1, 111.8)
- moved R1 1.64 mm to (108.6, 105.1)
- moved R3 1.64 mm to (118.6, 105.1)
- moved R5 1.64 mm to (131.2, 105.1)
- moved R6 1.64 mm to (136.3, 105.1)
- moved R7 1.64 mm to (141.4, 105.1)
- moved R8 1.64 mm to (146.3, 105.1)
- moved U3 1.64 mm to (161.4, 111.9)
- moved U4 1.64 mm to (184.0, 111.9)
- moved R10 1.64 mm to (158.9, 105.2)
- moved R12 1.64 mm to (169.0, 105.2)
- moved R14 1.64 mm to (181.5, 105.2)
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Connections:
- J2 pad 1: Net-(C1-Pad1) -> Net-(J2-Pin_1)
- J2 pad 2: Net-(C2-Pad1) -> Net-(J2-Pin_2)
- J2 pad 3: Net-(C3-Pad1) -> Net-(J2-Pin_3)
- J2 pad 4: Net-(C4-Pad1) -> Net-(J2-Pin_4)
- J3 pad 1: Net-(C5-Pad1) -> Net-(J3-Pin_1)
- J3 pad 2: Net-(C6-Pad1) -> Net-(J3-Pin_2)
- J3 pad 3: Net-(C7-Pad1) -> Net-(J3-Pin_3)
- J3 pad 4: Net-(C8-Pad1) -> Net-(J3-Pin_4)
- J4 pad 1: Net-(C9-Pad1) -> Net-(J4-Pin_1)
- J4 pad 2: Net-(C10-Pad1) -> Net-(J4-Pin_2)
- J4 pad 3: Net-(C11-Pad1) -> Net-(J4-Pin_3)
- J4 pad 4: Net-(C12-Pad1) -> Net-(J4-Pin_4)
- J5 pad 1: Net-(C13-Pad1) -> Net-(J5-Pin_1)
- J5 pad 2: Net-(C14-Pad1) -> Net-(J5-Pin_2)
- J5 pad 3: Net-(C15-Pad1) -> Net-(J5-Pin_3)
- J5 pad 4: Net-(C16-Pad1) -> Net-(J5-Pin_4)
- J7 pad MP: (no net) -> GND
- J8 pad MP: (no net) -> GND
Routing:
- net GND: track 4.56 -> 15.0 mm
- net Net-(J3-Pin_3): track 0.00 -> 7.85 mm
- net Net-(J3-Pin_2): track 0.00 -> 7.83 mm
- net Net-(J3-Pin_4): track 0.00 -> 7.81 mm
- net Net-(J2-Pin_4): track 0.00 -> 7.81 mm
- net Net-(J3-Pin_1): track 0.00 -> 7.81 mm
- net Net-(J2-Pin_3): track 0.00 -> 7.79 mm
- net Net-(J2-Pin_2): track 0.00 -> 7.78 mm
- net Net-(J2-Pin_1): track 0.00 -> 7.76 mm
- net Net-(J5-Pin_1): track 0.00 -> 7.68 mm
- net Net-(J4-Pin_1): track 0.00 -> 7.68 mm
- net Net-(J5-Pin_3): track 0.00 -> 7.67 mm
- net Net-(J4-Pin_3): track 0.00 -> 7.67 mm
- net Net-(J5-Pin_2): track 0.00 -> 7.65 mm
- net Net-(J4-Pin_2): track 0.00 -> 7.65 mm
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Other:
- board text added: "Optional series resistors for use with systems that can't handle the full 24v"
