File: SEM card breakout/SEM card breakout.kicad_pcb (KiCad board)
At the start: 2 copper layers, 254 x 345.4 mm, 4 parts, among them J1 SEM card edge connector, J2 SEM card edge connector, J3 Conn_02x25_Odd_Even, J4 Conn_02x25_Odd_Even

Commit message: tweaked dimensions
Parts:
- moved J1 8.50 mm to (73.9, 344.7)
- moved J2 8.50 mm to (73.9, -3.25)
- moved J4 8.50 mm to (34.3, 83.2)
- moved J3 8.50 mm to (34.4, 13.9)
Other:
- board size 254 x 345.4 mm -> 253.9 x 345.6 mm
- board text added: "Amray SEM card extender / diagnostic board"
- board text added: "Components on numbered side"
- board text added: "Solder on lettered side"
