File: Radio Shack Mini Speaker work-alike/Radio Shack Mini Speaker work-alike.kicad_sch (KiCad schematic)
At the start: 24 parts, among them J1 input, J2 aux speaker out, Q1 2SC1815, SW1 SW_SPDT, U1 LM386

Commit message: cleaned up for fab
Connections:
- net VCC: now also SW1.2 (B); no longer SW1.3 (C)
- net at BT1.1 (+): now also SW1.3 (C); no longer SW1.2 (B)
Other:
- moved on the sheet: SW1
Changed lines of the file:
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@@
+    (stroke (width 0) (type default))
+  )
+  (wire (pts (xy 153.035 83.185) (xy 156.845 83.185))
     (stroke (width 0) (type default))
   )
@@
     (stroke (width 0) (type default))
   )
-  (wire (pts (xy 156.845 111.76) (xy 156.845 78.105))
+  (wire (pts (xy 156.845 111.76) (xy 156.845 83.185))
     (stroke (width 0) (type default))
   )
@@
   )
   (wire (pts (xy 106.68 95.25) (xy 109.22 95.25))
-    (stroke (width 0) (type default))
-  )
-  (wire (pts (xy 156.845 78.105) (xy 153.035 78.105))
     (stroke (width 0) (type default))
   )
@@
     )
   )
-  (symbol (lib_id "Switch:SW_SPDT") (at 147.955 78.105 0) (mirror y) (unit 1)
-    (in_bom yes) (on_board yes) (dnp no) (fields_autoplaced)
-    (property "Reference" "SW1" (at 147.955 71.2175 0)
-      (effects (font (size 1.27 1.27)))
-    )
-    (property "Value" "SW_SPDT" (at 147.955 73.9926 0)
-      (effects (font (size 1.27 1.27)))
-    )
-    (property "Footprint" "Connector_PinHeader_2.54mm:PinHeader_1x03_P2.54mm_Vertical" (at 147.955 78.105 0)
-      (effects (font (size 1.27 1.27)) hide)
-    )
-    (property "Datasheet" "~" (at 147.955 78.105 0)
-      (effects (font (size 1.27 1.27)) hide)
-    )
+  (symbol (lib_id "Switch:SW_SPDT") (at 147.955 80.645 0) (unit 1)
+    (in_bom yes) (on_board yes) (dnp no)
+    (property "Reference" "SW1" (at 147.955 73.7575 0)
+      (effects (font (size 1.27 1.27)))
+    )
+    (property "Value" "SW_SPDT" (at 147.955 76.5326 0)
+      (effects (font (size 1.27 1.27)))
+    )
+    (property "Footprint" "Connector_PinHeader_2.54mm:PinHeader_1x03_P2.54mm_Vertical" (at 147.955 80.645 0)
+      (effects (font (size 1.27 1.27)) hide)
+    )
+    (property "Datasheet" "~" (at 147.955 80.645 0)
+      (effects (font (size 1.27 1.27)) hide)
+    )
