File: ascii to raw matrix/ascii to raw matrix.kicad_pcb (KiCad board)
At the start: 2 copper layers, 132.6 x 71.1 mm, 44 parts, among them J1 Conn_01x02_Pin, J10 parallel ascii, J11 apple 2e platinum, J2 Conn_01x02_Pin, J3 Conn_01x02_Pin, J4 Conn_01x02_Pin, J5 invert strobe, J6 invert busy, J7 reset, J8 power in, J9 parallel ascii, U1 74LS138, U2 74LS86, U3 74AHCT595, U4 74HCT597, U5 74HCT597, U6 Arduino Pro Mini, U7 L7805

Commit message: cleaned up for fab
Parts:
- added G***: LOGO, Evan's parts:pcbway logo, F.Cu at (202.6, 88.3)
